File: holo-video-player.kicad_sch (KiCad schematic)
At the start: 11 parts, among them J1 Conn_02x10_Odd_Even, J2 Conn_02x10_Odd_Even, J3 Conn_01x03_Pin, J4 Conn_01x03_Pin, U1 TLV493D, U2 AP2112K-3.3

Commit message: Adding JLCPCB Part Registrations.
Parts:
- C1: JLCPCB (none) -> C14663
- C2, C3: JLCPCB (none) -> C96446
- U1: JLCPCB (none) -> C126688
- U2: JLCPCB (none) -> C51118
Changed lines of the file:
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@@
 			)
 		)
-		(property "Datasheet" "~"
+		(property "Datasheet" "https://wmsc.lcsc.com/wmsc/upload/file/pdf/v2/lcsc/2211101700_YAGEO-CC0603KRX7R9BB104_C14663.pdf"
 			(at 58.42 27.94 0)
 			(effects
@@
 			)
 		)
-		(property "JLCPCB" ""
+		(property "JLCPCB" "C14663"
 			(at 58.42 27.94 0)
 			(effects
@@
 			)
 		)
-		(property "Datasheet" "~"
+		(property "Datasheet" "https://wmsc.lcsc.com/wmsc/upload/file/pdf/v2/lcsc/2304140030_Samsung-Electro-Mechanics-CL10A106MA8NRNC_C96446.pdf"
 			(at 46.99 27.94 0)
 			(effects
@@
 			)
 		)
-		(property "JLCPCB" ""
+		(property "JLCPCB" "C96446"
 			(at 46.99 27.94 0)
 			(effects
@@
 			)
 		)
-		(property "Datasheet" "~"
+		(property "Datasheet" "https://wmsc.lcsc.com/wmsc/upload/file/pdf/v2/lcsc/2304140030_Samsung-Electro-Mechanics-CL10A106MA8NRNC_C96446.pdf"
 			(at 16.51 27.94 0)
 			(effects
@@
 			)
 		)
-		(property "JLCPCB" ""
+		(property "JLCPCB" "C96446"
 			(at 16.51 27.94 0)
 			(effects
@@
 			)
 		)
-		(property "JLCPCB" ""
+		(property "JLCPCB" "C126688"
 			(at 87.63 30.48 0)
 			(effects
@@
 			)
 		)
-		(property "JLCPCB" ""
+		(property "JLCPCB" "C51118"
 			(at 33.02 25.4 0)
 			(effects
